Commit message: E2: feat: camera evidence baseline — pitched front camera, matte road materials, lane-line visibility verified
feat: verify the ZEDm front camera publishes headless (640x480 RGB @ 20 Hz,
bridged camera/image_raw) and capture frame evidence at four canonical poses
(experiments/sim/e_cam_visibility).

fix: pitch the camera down 0.25 rad in both gazebo URDFs — flat-mounted, the
R=0.80 m curve swept out of the FOV at curve entry.

fix: matte road tiles (roughness 0.9, metalness 0.0) in compose_lane_circuit's
material template; ogre2 PBR defaults rendered glossy specular lobes a
white-line detector / CNN would read as lane features. All three oval worlds
regenerated (content-identical otherwise; centerline byte-identical; wet/worn
lose accidental CRLF endings).

chore: add tools/capture_camera_frames.py, tools/cam_evidence_session.sh,
tools/reap_sim.sh.

Verification: pytest 366 passed; check_traceability PASS; evidence frames
reviewed for flat vs pitched vs pitched+matte.

Co-Authored-By: Claude Fable 5 <noreply@anthropic.com>

File: src/cobraflex/urdf/my_robot_gazebo.urdf (robot description, URDF)
Before this commit: robot cobraflex_robot, 7 links, 6 joints
Joints:
- joint camera_joint: origin xyz=${body_length/2} 0 0.02 rpy=0 0 0 -> xyz=${body_length/2} 0 0.02 rpy=0 0.25 0

File: src/cobraflex/urdf/my_robot_gazebo_mesh.urdf (robot description, URDF)
Before this commit: robot cobraflex_robot, 7 links, 6 joints
Joints:
- joint camera_joint: origin xyz=${body_length/2 - 0.04} 0 0.02 rpy=0 0 0 -> xyz=${body_length/2 - 0.04} 0 0.02 rpy=0 0.25 0
