Commit message: E4: Migration to Isaac Sim

File: src/cobraflex/urdf/my_robot_gazebo.urdf (robot description, URDF)
Before this commit: robot cobraflex_robot, 9 links, 8 joints
Joints:
- joint camera_joint: origin xyz=${body_length/2} 0 0.02 rpy=0 0.25 0 -> xyz=${body_length/2} 0 0.02 rpy=0 0 0

File: src/cobraflex/urdf/my_robot_gazebo_mesh.urdf (robot description, URDF)
Before this commit: robot cobraflex_robot, 9 links, 8 joints
Joints:
- joint camera_joint: origin xyz=${body_length/2 - 0.04} 0 0.02 rpy=0 0.25 0 -> xyz=${body_length/2 - 0.0475} 0 0.02 rpy=0 0 0
- joint imu_joint: origin xyz=${body_length/2 - 0.04} 0 0.02 rpy=0 0 0 -> xyz=${body_length/2 - 0.0475} 0 0.02 rpy=0 0 0

File: src/cobraflex/urdf/my_robot_mesh.urdf (robot description, URDF)
Before this commit: robot cobraflex_robot, 10 links, 9 joints
Joints:
- joint camera_joint: origin xyz=${body_length/2 - 0.04} 0 0.02 rpy=0 0 0 -> xyz=${body_length/2 - 0.0475} 0 0.02 rpy=0 0 0
- joint imu_joint: origin xyz=${body_length/2 - 0.04} 0 0.02 rpy=0 0 0 -> xyz=${body_length/2 - 0.0475} 0 0.02 rpy=0 0 0

Commit message: E4: Implement domain randomization features in IsaacSim training, including dynamics and scene randomization, and update camera frame ID for lane keeping.

File: src/cobraflex/urdf/my_robot_gazebo.urdf (robot description, URDF)
Before this commit: robot cobraflex_robot, 9 links, 8 joints
Links:
- removed link camera_link
- removed link camera_link_optical
- link camera_link_lane: geometry collision cylinder length=0.002 radius=0.005; visual cylinder length=0.002 radius=0.005
Joints:
- removed joint camera_joint
- removed joint camera_optical_joint
- added joint zedm_mount_joint: type fixed, parent body_link, child zedm_camera_link, origin xyz=${body_length/2 - 0.0475} 0 ${0.02 - 0.0265/2} rpy=0 0 0

File: src/cobraflex/urdf/my_robot_mesh.urdf (robot description, URDF)
Before this commit: robot cobraflex_robot, 10 links, 9 joints
Links:
- link camera_link_lane: geometry collision cylinder length=0.002 radius=0.005; visual cylinder length=0.002 radius=0.005
