Commit message: E4: Add lane camera support and update related configurations
- Introduced a new camera link and joint in URDF files for lane camera integration.
- Updated Gazebo simulation files to include the lane camera sensor with appropriate parameters.
- Adjusted camera height in URDF to account for new mounting position.
- Modified camera geometry calculations in Python to reflect new camera specifications.
- Updated CV lane estimator node to subscribe to the new lane camera topic.
- Changed evaluation and training scripts to use the lane camera topic for observations.
- Enhanced training configuration to specify lane camera topic.
- Updated cleanup script to ensure proper termination of lane estimator processes.

File: src/cobraflex/urdf/my_robot_basic.urdf (robot description, URDF)
Before this commit: robot cobraflex_robot, 7 links, 7 joints
Links:
- added link camera_link_lane; collision box size=0.005 0.02 0.02; visual box size=0.005 0.02 0.02
- added link camera_link_optical_lane
Joints:
- added joint camera_joint_lane: type fixed, parent body_link, child camera_link_lane, origin xyz=${body_length/2 + 0.01} 0 -0.03 rpy=0 0.3 0
- added joint camera_optical_joint_lane: type fixed, parent camera_link_lane, child camera_link_optical_lane, origin xyz=0 0 0 rpy=${-pi/2} 0 ${-pi/2}

File: src/cobraflex/urdf/my_robot_gazebo.urdf (robot description, URDF)
Before this commit: robot cobraflex_robot, 7 links, 6 joints
Links:
- added link camera_link_lane; collision box size=0.005 0.02 0.02; visual box size=0.005 0.02 0.02
- added link camera_link_optical_lane
Joints:
- added joint camera_joint_lane: type fixed, parent body_link, child camera_link_lane, origin xyz=${body_length/2 + 0.01} 0 -0.03 rpy=0 0.30 0
- added joint camera_optical_joint_lane: type fixed, parent camera_link_lane, child camera_link_optical_lane, origin xyz=0 0 0 rpy=${-pi/2} 0 ${-pi/2}

File: src/cobraflex/urdf/my_robot_gazebo_mesh.urdf (robot description, URDF)
Before this commit: robot cobraflex_robot, 7 links, 6 joints
Links:
- added link camera_link_lane; collision box size=0.005 0.02 0.02; visual box size=0.005 0.02 0.02
- added link camera_link_optical_lane
Joints:
- added joint camera_joint_lane: type fixed, parent body_link, child camera_link_lane, origin xyz=${body_length/2 + 0.01} 0 -0.03 rpy=0 0.30 0
- added joint camera_optical_joint_lane: type fixed, parent camera_link_lane, child camera_link_optical_lane, origin xyz=0 0 0 rpy=${-pi/2} 0 ${-pi/2}
- joint body_joint: origin xyz=0 0 ${body_height/2 + chassis_height/2} -> xyz=0 0 ${body_height/2 + chassis_height/2 - 0.01}

File: src/cobraflex/urdf/my_robot_mesh.urdf (robot description, URDF)
Before this commit: robot cobraflex_robot, 8 links, 7 joints
Links:
- added link camera_link_lane; collision box size=0.005 0.02 0.02; visual box size=0.005 0.02 0.02
- added link camera_link_optical_lane
Joints:
- added joint camera_joint_lane: type fixed, parent body_link, child camera_link_lane, origin xyz=${body_length/2 + 0.01} 0 -0.03 rpy=0 0.30 0
- added joint camera_optical_joint_lane: type fixed, parent camera_link_lane, child camera_link_optical_lane, origin xyz=0 0 0 rpy=${-pi/2} 0 ${-pi/2}
- joint body_joint: origin xyz=0 0 ${body_height/2 + chassis_height/2} -> xyz=0 0 ${body_height/2 + chassis_height/2 - 0.01}
