Commit message: E5: Sim2Real deploy

File: src/cobraflex/urdf/my_robot_basic.urdf (robot description, URDF)
Before this commit: robot cobraflex_robot, 9 links, 9 joints
Links:
- added link viz_bumpers; visual box size=0.020 0.116 0.020; visual box size=0.022 0.124 0.020
- added link viz_chassis_rails; visual box size=0.170 0.020 0.034; visual box size=0.170 0.020 0.034
- added link viz_deck_hardware; visual box size=0.082 0.082 0.014; visual cylinder length=0.086 radius=0.0035
- added link viz_drivetrain; visual cylinder length=0.049 radius=0.006; visual cylinder length=0.049 radius=0.006
- added link viz_jetson; visual box size=0.105 0.092 0.043
- added link viz_lane_cam_lens; visual cylinder length=0.001 radius=0.0034; visual cylinder length=0.009 radius=0.0055
- added link viz_lidar_aperture; visual box size=0.012 0.024 0.013
- added link viz_lidar_head; visual cylinder length=0.018 radius=0.0350
- added link viz_lidar_standoffs; visual cylinder length=0.020 radius=0.003; visual cylinder length=0.020 radius=0.003
- added link viz_lipo; visual box size=0.078 0.046 0.028
- added link viz_mast_plate; visual box size=0.014 0.100 0.008
- added link viz_motor; visual cylinder length=0.048 radius=0.0165
- added link viz_servo; visual box size=0.040 0.021 0.037
- added link viz_skirts; visual box size=0.190 0.008 0.048; visual box size=0.190 0.008 0.048
- link base_link: geometry collision box size=${chassis_length} ${chassis_width} ${chassis_height}; visual box size=${chassis_length} 0.112 0.010
- link body_link: geometry collision box size=${body_length} ${body_width} ${body_height}; visual box size=${body_length} 0.176 0.008
- link camera_link: geometry collision box size=0.01 0.1 0.02
- link camera_link_lane: geometry collision box size=0.005 0.02 0.02; visual box size=0.004 0.025 0.024
- link lidar_link: geometry collision cylinder length=0.04 radius=0.0375; visual cylinder length=0.012 radius=0.0375
Joints:
- added joint viz_bumpers_joint: type fixed, parent base_link, child viz_bumpers, origin xyz=0 0 0 rpy=0 0 0
- added joint viz_chassis_rails_joint: type fixed, parent base_link, child viz_chassis_rails, origin xyz=0 0 0 rpy=0 0 0
- added joint viz_deck_hardware_joint: type fixed, parent body_link, child viz_deck_hardware, origin xyz=0 0 0 rpy=0 0 0
- added joint viz_drivetrain_joint: type fixed, parent base_link, child viz_drivetrain, origin xyz=0 0 0 rpy=0 0 0
- added joint viz_jetson_joint: type fixed, parent body_link, child viz_jetson, origin xyz=0 0 0 rpy=0 0 0
- added joint viz_lane_cam_lens_joint: type fixed, parent camera_link_lane, child viz_lane_cam_lens, origin xyz=0 0 0 rpy=0 0 0
- added joint viz_lidar_aperture_joint: type fixed, parent lidar_link, child viz_lidar_aperture, origin xyz=0 0 0 rpy=0 0 0
- added joint viz_lidar_head_joint: type fixed, parent lidar_link, child viz_lidar_head, origin xyz=0 0 0 rpy=0 0 0
- added joint viz_lidar_standoffs_joint: type fixed, parent lidar_link, child viz_lidar_standoffs, origin xyz=0 0 0 rpy=0 0 0
- added joint viz_lipo_joint: type fixed, parent body_link, child viz_lipo, origin xyz=0 0 0 rpy=0 0 0
- added joint viz_mast_plate_joint: type fixed, parent body_link, child viz_mast_plate, origin xyz=0 0 0 rpy=0 0 0
- added joint viz_motor_joint: type fixed, parent base_link, child viz_motor, origin xyz=0 0 0 rpy=0 0 0
- added joint viz_servo_joint: type fixed, parent base_link, child viz_servo, origin xyz=0 0 0 rpy=0 0 0
- added joint viz_skirts_joint: type fixed, parent body_link, child viz_skirts, origin xyz=0 0 0 rpy=0 0 0

File: src/cobraflex/urdf/zed_descr.urdf.xacro (robot description, xacro)
@@ -10,5 +10,9 @@
   <xacro:arg name="gnss_z" default="0.0" />
   <xacro:include filename="$(find cobraflex)/urdf/zed_macro.urdf.xacro" />
-  <xacro:zed_camera name="$(arg camera_name)" model="$(arg camera_model)" custom_baseline="$(arg custom_baseline)" enable_gnss="$(arg enable_gnss)">
+  <!-- This wrapper is included ONLY by my_robot_basic.urdf, the RViz/hardware
+       description. mat_override lifts the zedm shell off rgba 0,0,0, which
+       RViz shades to an unlit void at the very front of the robot. The Gazebo
+       URDFs include zed_macro directly and so keep the stock colour. -->
+  <xacro:zed_camera name="$(arg camera_name)" model="$(arg camera_model)" custom_baseline="$(arg custom_baseline)" enable_gnss="$(arg enable_gnss)" mat_override="0.22 0.23 0.27 1.0">
 	    <origin xyz="$(arg gnss_x) $(arg gnss_y) $(arg gnss_z)" rpy="0 0 0"/>
   </xacro:zed_camera>

File: src/cobraflex/urdf/zed_macro.urdf.xacro (robot description, xacro)
@@ -23,5 +23,12 @@
       - enable_gnss: if true enable the URDF link
   -->
-  <xacro:macro name="zed_camera" params="name=zed model=zed enable_gnss=false custom_baseline=0 *gnss_origin">
+  <!-- mat_override: optional rgba replacing the per-model shell colour. The
+       default sentinel 'none' keeps every existing caller byte-identical -
+       my_robot_gazebo.urdf and my_robot_gazebo_mesh.urdf must NOT change,
+       because their cameras render this mesh and they are the models behind
+       the recorded campaign evidence. Only zed_descr.urdf.xacro (RViz /
+       hardware description) passes it, to lift the zedm shell off rgba 0,0,0,
+       which RViz shades to an unlit void. -->
+  <xacro:macro name="zed_camera" params="name=zed model=zed enable_gnss=false custom_baseline=0 mat_override=none *gnss_origin">
     <xacro:if value="${model == 'zed'}">
       <xacro:property name="baseline" value="0.12" />
@@ -153,4 +160,7 @@
       <xacro:property name="mono" value="true" />
       <xacro:property name="mat" value="0.25 0.25 0.25 1.0" />
+    </xacro:if>
+    <xacro:if value="${mat_override != 'none'}">
+      <xacro:property name="mat" value="${mat_override}" />
     </xacro:if>
     <!-- Camera mounting point (the threaded screw hole in the bottom) -->

Commit message: E5: Sim2Real deploy

File: src/cobraflex/urdf/my_robot_basic.urdf (robot description, URDF)
Before this commit: robot cobraflex_robot, 23 links, 23 joints
Joints:
- removed joint footprint_joint
- added joint zed_mount_joint: type fixed, parent body_link, child zed_camera_link, origin xyz=0.11 0 0.02 rpy=0 0 0
