Commit message: ZED cameras update

File: src/cobraflex/urdf/my_robot_gazebo_mesh.urdf (robot description, URDF)
Before this commit: robot cobraflex_robot, 9 links, 8 joints
Links:
- removed link camera_link
- removed link camera_link_optical
Joints:
- removed joint camera_joint
- removed joint camera_optical_joint
- added joint zedm_mount_joint: type fixed, parent body_link, child zedm_camera_link, origin xyz=${body_length/2 - 0.0475} 0 ${0.02 - 0.0265/2} rpy=0 0 0

File: src/cobraflex/urdf/zed_macro.urdf.xacro (robot description, xacro)
@@ -205,5 +205,5 @@
         <parent link="${name}_camera_center"/>
         <child link="${name}_left_camera_frame"/>
-        <origin xyz="${optical_offset_x} ${baseline/2} 0" rpy="0 0 0" />
+        <origin xyz="${optical_offset_x + 0.02} ${baseline/2 - 0.007} 0" rpy="0 0 0" />
       </joint>
       <link name="${name}_left_camera_frame_optical"/>
@@ -236,5 +236,5 @@
         <parent link="${name}_camera_center"/>
         <child link="${name}_right_camera_frame"/>
-        <origin xyz="${optical_offset_x} -${baseline/2} 0" rpy="0 0 0" />
+        <origin xyz="${optical_offset_x + 0.02} -${baseline/2 + 0.007} 0" rpy="0 0 0" />
       </joint>
       <link name="${name}_right_camera_frame_optical"/>
