Commit message: E5: Sim2Real stl files

File: src/cobraflex/urdf/my_robot_gazebo_mesh.urdf (robot description, URDF)
Before this commit: robot cobraflex_robot, 7 links, 7 joints
Joints:
- joint camera_joint_lane: origin xyz=${body_length/2 + 0.01} 0 -0.03 rpy=0 0.30 0 -> xyz=${body_length/2 + 0.02} 0 -0.03 rpy=0 0 0

Commit message: E5: URDF Update

File: src/cobraflex/urdf/my_robot_gazebo_mesh.urdf (robot description, URDF)
Before this commit: robot cobraflex_robot, 7 links, 7 joints
Joints:
- joint body_joint: origin xyz=0 0 ${body_height/2 + chassis_height/2 - 0.01} -> xyz=0 0 ${body_height/2 + chassis_height/2 - 0.005}
- joint camera_joint_lane: origin xyz=${body_length/2 + 0.02} 0 -0.03 rpy=0 0 0 -> xyz=${body_length/2 + 0.018} -0.0015 -0.026 rpy=0 0 0
