Commit message: E4: Migration to Isaac Sim

File: src/cobraflex/urdf/cobraflex_isaac.urdf (robot description, URDF)
Before this commit: robot cobraflex_robot, 13 links, 12 joints
Links:
- removed link camera_link
- removed link camera_link_optical
- added link zedm_camera_center; collision mesh filename=../meshes/zedmini_camera.stl scale=0.001 0.001 0.001; visual mesh filename=../meshes/zedmini_camera.stl scale=0.001 0.001 0.001
- added link zedm_camera_link
- added link zedm_left_camera_frame
- added link zedm_left_camera_frame_optical
- added link zedm_right_camera_frame
- added link zedm_right_camera_frame_optical
Joints:
- removed joint camera_joint
- removed joint camera_optical_joint
- added joint zedm_camera_center_joint: type fixed, parent zedm_camera_link, child zedm_camera_center, origin xyz=0 0 0.01325 rpy=0 0 0
- added joint zedm_left_camera_joint: type fixed, parent zedm_camera_center, child zedm_left_camera_frame, origin xyz=0.02 0.0245 0 rpy=0 0 0
- added joint zedm_left_camera_joint_optical: type fixed, parent zedm_left_camera_frame, child zedm_left_camera_frame_optical, origin xyz=0 0 0 rpy=-1.5707963267948966 0.0 -1.5707963267948966
- added joint zedm_mount_joint: type fixed, parent body_link, child zedm_camera_link, origin xyz=0.0665 0 0.00675 rpy=0 0 0
- added joint zedm_right_camera_joint: type fixed, parent zedm_camera_center, child zedm_right_camera_frame, origin xyz=0.02 -0.0385 0 rpy=0 0 0
- added joint zedm_right_camera_joint_optical: type fixed, parent zedm_right_camera_frame, child zedm_right_camera_frame_optical, origin xyz=0 0 0 rpy=-1.5707963267948966 0.0 -1.5707963267948966

Commit message: E4: Migration to Isaac Sim

File: src/cobraflex/urdf/cobraflex_isaac.urdf (robot description, URDF)
Before this commit: robot cobraflex_robot, 17 links, 16 joints
Links:
- link camera_link_lane: geometry collision cylinder length=0.002 radius=0.005; visual cylinder length=0.002 radius=0.005
Joints:
- joint zedm_camera_center_joint: origin xyz=0 0 0.01325 rpy=0 0 0 -> xyz=0 0 0.01325 rpy=0 0.0 0
- joint zedm_mount_joint: origin xyz=0.0665 0 0.00675 rpy=0 0 0 -> xyz=0.0665 0 0.006750000000000001 rpy=0 0 0

File: src/cobraflex/urdf/my_robot_gazebo_mesh.urdf (robot description, URDF)
Before this commit: robot cobraflex_robot, 7 links, 7 joints
Links:
- link camera_link_lane: geometry collision cylinder length=0.002 radius=0.005; visual cylinder length=0.002 radius=0.005
