Commit message: E5: Sim2Real

File: src/cobraflex/urdf/cobraflex_isaac.urdf (robot description, URDF)
Before this commit: robot cobraflex_robot, 17 links, 16 joints
Links:
- link base_link: mass 5.0 -> 2.0172
- link body_link: mass 1.0 -> 0.8928

Commit message: E5: URDF Update

File: src/cobraflex/urdf/cobraflex_isaac.urdf (robot description, URDF)
Before this commit: robot cobraflex_robot, 17 links, 16 joints
Joints:
- joint body_joint: origin xyz=0 0 0.07 -> xyz=0 0 0.075
- joint camera_joint_lane: origin xyz=0.124 0 -0.03 rpy=0 0.30 0 -> xyz=0.132 -0.0015 -0.03431 rpy=0 0.31132 0
- joint zedm_mount_joint: origin xyz=0.0665 0 0.006750000000000001 rpy=0 0 0 -> xyz=0.07050000000000001 -0.0015 0.011750000000000002 rpy=0 0 0

File: src/cobraflex/urdf/my_robot_basic.urdf (robot description, URDF)
Before this commit: robot cobraflex_robot, 23 links, 23 joints
Joints:
- joint body_joint: origin xyz=0 0 ${body_height/2 + chassis_height/2} -> xyz=0 0 ${body_height/2 + chassis_height/2 - 0.005}
- joint camera_joint_lane: origin xyz=${body_length/2 + 0.01} 0 -0.03 rpy=0 0.3 0 -> xyz=${body_length/2 + 0.018} -0.0015 -0.03431 rpy=0 0.31132 0

File: src/cobraflex/urdf/my_robot_gazebo.urdf (robot description, URDF)
Before this commit: robot cobraflex_robot, 7 links, 7 joints
Joints:
- joint body_joint: origin xyz=0 0 ${body_height/2 + chassis_height/2} -> xyz=0 0 ${body_height/2 + chassis_height/2 - 0.005}
- joint camera_joint_lane: origin xyz=${body_length/2 + 0.01} 0 -0.03 rpy=0 0.30 0 -> xyz=${body_length/2 + 0.018} -0.0015 -0.03431 rpy=0 0.31132 0

File: src/cobraflex/urdf/my_robot_gazebo_mesh.urdf (robot description, URDF)
Before this commit: robot cobraflex_robot, 7 links, 7 joints
Joints:
- joint camera_joint_lane: origin xyz=${body_length/2 + 0.018} -0.0015 -0.026 rpy=0 0 0 -> xyz=${body_length/2 + 0.018} -0.0015 -0.03431 rpy=0 0.31132 0
- joint zedm_mount_joint: origin xyz=${body_length/2 - 0.0475} 0 ${0.02 - 0.0265/2} rpy=0 0 0 -> xyz=${body_length/2 - 0.0435} -0.0015 ${0.025 - 0.0265/2} rpy=0 0 0

File: src/cobraflex/urdf/my_robot_mesh.urdf (robot description, URDF)
Before this commit: robot cobraflex_robot, 10 links, 9 joints
Joints:
- joint body_joint: origin xyz=0 0 ${body_height/2 + chassis_height/2 - 0.01} -> xyz=0 0 ${body_height/2 + chassis_height/2 - 0.005}
- joint camera_joint: origin xyz=${body_length/2 - 0.0475} 0 0.02 rpy=0 0 0 -> xyz=${body_length/2 - 0.0435} -0.0015 ${0.035 - 0.0265/2} rpy=0 0 0
- joint camera_joint_lane: origin xyz=${body_length/2 + 0.01} 0 -0.03 rpy=0 0.30 0 -> xyz=${body_length/2 + 0.018} -0.0015 -0.03431 rpy=0 0.31132 0
